Commit message: Add optical camera link

File: urdf/kinect_robot.xacro (robot description, xacro)
@@ -147,4 +147,11 @@
     <axis xyz="0 1 0" rpy="0 0 0"/>
   </joint>
+  <link name="camera_link_optical">
+  </link>
+  <joint name="camera_optical_joint" type="fixed">
+    <origin xyz="0 0 0" rpy="-1.5707 0 -1.5707"/>
+    <parent link="camera_link"/>
+    <child link="camera_link_optical"/>
+  </joint>
   <link name='hokuyo'>
     <inertial>

Commit message: Fix references to camera link and .gazebo in kinect_robot.xacro

File: urdf/kinect_robot.xacro (robot description, xacro)
@@ -1,5 +1,5 @@
 <?xml version='1.0'?>
 <robot name="simple_robot" xmlns:xacro="http://www.ros.org/wiki/xacro">
-  <xacro:include filename="$(find my_robot_world)/urdf/simple_robot.gazebo" />
+  <xacro:include filename="$(find my_robot_world)/urdf/kinect_robot.gazebo" />
   <link name="robot_footprint"></link>
   <joint name="robot_footprint_joint" type="fixed">
@@ -151,5 +151,5 @@
   <joint name="camera_optical_joint" type="fixed">
     <origin xyz="0 0 0" rpy="-1.5707 0 -1.5707"/>
-    <parent link="camera_link"/>
+    <parent link="camera"/>
     <child link="camera_link_optical"/>
   </joint>

Commit message: Different colors for kinect_robot

File: urdf/kinect_robot.xacro (robot description, xacro)
@@ -184,11 +184,11 @@
   </joint>
   <gazebo reference="left_wheel">
-    <material>Gazebo/Green</material>
+    <material>Gazebo/SkyBlue</material>
   </gazebo>
   <gazebo reference="right_wheel">
-    <material>Gazebo/Green</material>
+    <material>Gazebo/SkyBlue</material>
   </gazebo>
   <gazebo reference="chassis">
-    <material>Gazebo/SkyBlue</material>
+    <material>Gazebo/DarkGrey</material>
   </gazebo>
   <gazebo reference="camera">
